File: DoorButtonBoard.kicad_pcb (KiCad board)
At the start: 2 copper layers, 57.2 x 38.1 mm, 16 parts, among them J1 Conn_01x04, J2 Conn_01x02, J3 Conn_01x04, SW1 SW_Push, U1 APA102C, U2 APA102C, U3 APA102C

Commit message: Finish Rev A
Parts:
- moved C1 71.5 mm to (121.0, 91.2)
- moved C2 65.2 mm to (139.2, 95.0)
- moved R3 52.1 mm to (137.8, 108.0), turned to 90 degrees
- moved R2 14.7 mm to (132.2, 108.0), turned to 270 degrees
- moved R1 13.2 mm to (127.0, 108.0), turned to 90 degrees
- moved SW1 3.14 mm to (126.2, 95.8), turned to 45 degrees
- moved U3 1.96 mm to (121.0, 100.5)
- moved U2 1.88 mm to (139.3, 100.6)
Routing:
- net GND: track 0.00 -> 40.7 mm, vias 0 -> 7
- net Net-(J2-Pad1): track 0.00 -> 39.9 mm, vias 0 -> 2
- net Net-(U1-Pad5): track 0.00 -> 33.0 mm
- net Net-(U1-Pad6): track 0.00 -> 26.8 mm
- net +5V: track 0.00 -> 26.1 mm
- net Net-(R1-Pad2): track 0.00 -> 23.4 mm, vias 0 -> 2
- net /DI: track 0.00 -> 21.1 mm
- net /CI: track 0.00 -> 21.0 mm
- net Net-(U2-Pad5): track 0.00 -> 14.1 mm
- net Net-(U2-Pad6): track 0.00 -> 13.9 mm
- net /CO: track 0.00 -> 12.7 mm
- net /DO: track 0.00 -> 12.6 mm
- added copper zone on F.Cu, net +5V
- added copper zone on B.Cu, net GND
Other:
- board text added: "BUTTON"
- board text added: "Door Button Board - Rev A"
- board text added: "LED IN"
- board text added: "LED OUT"
- board text added: "Veenema Design Works (2018)"
